File: HandHeldDMM-main/DMM.kicad_pcb (KiCad board)
At the start: 2 copper layers, 60 x 100 mm, 162 parts, among them IC1 REF35300QDBVR, J1 Conn_02x03_Odd_Even, J2 Conn_01x02, J3 Conn_01x03, J4 Conn_02x05_Odd_Even, J5 Conn_01x02, J6 Conn_01x04, J7 Conn_01x02, J8 Conn_01x01, J9 Conn_01x01, Q1 HD6362, Q10 SI2301, Q11 SI2301, Q12 SI2301, Q2 HD6362, Q3 SI2302, Q4 SI2302, Q5 SI2302, Q6 SI2301, Q7 SI2301, Q8 HD6362, Q9 SI2301, SW1 SW_Push, U1 TLP291, U10 TLP291, U11 LM334M, U12 XC62KN33302PR-G, U13 CPC1017N, U14 CPC1017N, U15 CPC1017N, U16 CPC1017N, U17 TLP291, U18 TLP291, U19 TLP291, U2 LM358, U20 TLP291, U21 TLP291, U22 OPA2140, U3 TLP291, U4 TLP291, U5 OPA2140, U6 TLP291, U7 STM32F373CCTx, U8 AMS1117-3.3, U9 TLP291, Y1 16Mhz

Commit message: PCB work
Parts:
- moved R27 60.0 mm to (135.0, 115.6), turned to 90 degrees
- moved R25 57.6 mm to (135.0, 110.6), turned to 90 degrees
- moved R59 56.5 mm to (169.9, 69.8), turned to 0 degrees
- moved R13 56.0 mm to (135.0, 105.6), turned to 90 degrees
- moved R19 55.3 mm to (135.0, 100.6), turned to 90 degrees
- moved U14 54.0 mm to (139.9, 116.1), turned to 0 degrees
- moved Q12 53.9 mm to (169.9, 72.8), turned to -90 degrees
- moved U15 51.4 mm to (139.8, 111.1), turned to 0 degrees
- moved R56 51.0 mm to (166.1, 69.8), turned to 0 degrees
- moved R44 50.4 mm to (170.7, 76.6), turned to 0 degrees
- moved R39 49.9 mm to (170.7, 75.4)
- moved U13 49.5 mm to (139.8, 106.1), turned to 0 degrees
- moved U16 48.5 mm to (139.8, 101.1), turned to 0 degrees
- moved Q10 48.3 mm to (166.1, 72.8), turned to -90 degrees
- moved R48 47.5 mm to (168.8, 77.2), turned to 90 degrees
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Routing:
- net /Measurement Analog/1V: track 59.4 -> 6.58 mm, vias 2 -> 0
- net /Measurement Analog/10V: track 55.5 -> 6.57 mm, vias 2 -> 0
- net /Measurement Analog/100V: track 50.6 -> 6.58 mm, vias 2 -> 0
- net Net-(Q12-G): track 47.1 -> 5.35 mm
- net /Measurement Analog/1000V: track 45.6 -> 6.48 mm, vias 2 -> 0
- net Net-(Q10-G): track 44.0 -> 7.26 mm
- net Net-(Q9-G): track 41.0 -> 7.06 mm
- net Net-(Q7-G): track 38.0 -> 6.90 mm
- net GNDA: track 55.5 -> 25.3 mm, vias 12 -> 0
- net InputPosRaw: track 25.3 -> 0.00 mm
- net Net-(Q11-G): track 31.5 -> 6.83 mm
- net InputPos: track 117.8 -> 93.2 mm
- net Net-(Q6-G): track 25.7 -> 1.87 mm
- net +3.3V: track 22.2 -> 0.00 mm
- net InputAmps: track 70.1 -> 91.1 mm
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- removed copper zone on B.Cu, net GNDA

Commit message: More pcb work
Parts:
- R24, R28, R29, R63, R70: footprint Resistor_SMD:R_0402_1005Metric_Pad0.72x0.64mm_HandSolder -> Resistor_SMD:R_0603_1608Metric_Pad0.98x0.95mm_HandSolder
- moved J1 18.9 mm to (161.1, 32.5)
- moved J6 13.5 mm to (146.0, 30.8)
- moved U4 10.1 mm to (181.3, 67.7)
- moved U10 9.94 mm to (191.5, 67.7)
- moved R5 9.75 mm to (181.5, 62.3)
- moved R8 9.60 mm to (191.2, 62.2)
- moved R1 8.10 mm to (181.8, 35.6), turned to 90 degrees
- moved R63 7.92 mm to (175.4, 70.9)
- moved R3 7.42 mm to (181.8, 31.8), turned to 90 degrees
- moved R52 6.84 mm to (163.1, 56.9)
- moved U17 6.84 mm to (163.0, 61.9)
- moved U19 6.80 mm to (156.2, 61.9)
- moved R58 6.77 mm to (156.2, 56.9)
- moved JP1 6.64 mm to (168.6, 38.2), turned to 0 degrees
- moved C19 6.54 mm to (179.8, 29.6), turned to 180 degrees
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Routing:
- net GPIO_1: track 0.00 -> 83.9 mm
- net GPIO_2: track 0.00 -> 78.5 mm
- net GPIO_3: track 0.00 -> 72.3 mm
- net GPIO_4: track 0.00 -> 68.0 mm
- net SD-ADC1: track 0.00 -> 56.7 mm
- net NRST: track 0.00 -> 52.7 mm, vias 0 -> 1
- net BattOut+: track 0.00 -> 42.5 mm
- net GPIO_5: track 7.86 -> 44.5 mm
- net GPIO_7: track 14.6 -> 49.2 mm
- net InputAmps: track 91.1 -> 59.3 mm
- net GPIO_9: track 9.71 -> 41.3 mm
- net GPIO_10: track 0.00 -> 31.0 mm, vias 0 -> 2
- net SWCLK: track 0.00 -> 29.8 mm
- net GPIO_6: track 17.4 -> 46.4 mm
- net BattOut-: track 0.00 -> 28.5 mm
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- added copper zone on F.Cu, net GND
- added copper zone on F.Cu, net GNDA
Other:
- outline, holes or cut-outs redrawn
- board text added: "BOOT SELECT"
- board text added: "FIX ground fills and find good connection point' -weird islands -large single enged connections -power planes -back layer (power or gnd??)"
- board text removed: "Put unput Jacks on bottom and give more mov space??"
- board text removed: "To-do: - Using 3V Ref on analog side, what ground ref??? - also needed for ADC"

Commit message: PCB rev 1 with schematic change ideas
Parts:
- R10: footprint Resistor_THT:R_Axial_DIN0516_L15.5mm_D5.0mm_P7.62mm_Vertical -> Resistor_THT:R_Axial_DIN0516_L15.5mm_D5.0mm_P20.32mm_Horizontal
- moved R10 12.6 mm to (164.7, 105.5)
- moved C34 1.36 mm to (151.8, 35.3), turned to 0 degrees
- moved R21 0.95 mm to (177.9, 80.0)
- moved R4 0.90 mm to (177.3, 62.3)
- moved Q4 0.81 mm to (177.9, 83.0)
- moved R5 0.65 mm to (180.8, 62.3)
- moved R6 0.60 mm to (184.1, 62.3)
- moved R7 0.60 mm to (187.6, 62.2)
- moved U10 0.54 mm to (190.9, 67.7)
- moved U4 0.54 mm to (180.7, 67.7)
- moved U6 0.54 mm to (184.1, 67.7)
- moved U9 0.54 mm to (187.5, 67.7)
- moved R63 0.54 mm to (174.9, 70.9)
- moved U3 0.54 mm to (177.3, 67.7)
- moved R3 0.41 mm to (181.4, 31.9)
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Routing:
- net +3.3V: track 23.5 -> 162.6 mm, vias 0 -> 4
- net GNDA: track 8.30 -> 46.6 mm, vias 1 -> 58
- net GND: track 0.00 -> 5.63 mm, vias 0 -> 71
- net InputAmps: track 59.3 -> 54.6 mm
- net BattOut+: track 42.5 -> 46.4 mm
- net CurrentOut: track 14.0 -> 10.5 mm
- net InputPosRaw: track 26.5 -> 23.6 mm
- net Net-(Q1-G): track 47.8 -> 49.8 mm
- net Net-(D2-K): track 0.00 -> 1.81 mm
- net Net-(IC1-EN): track 6.74 -> 5.14 mm
- net GPIO_5: track 44.5 -> 43.4 mm
- net Net-(U22A-+): track 18.0 -> 18.8 mm
- net BattOut-: track 28.5 -> 29.2 mm
- net Net-(Q3-G): track 45.2 -> 44.6 mm
- net Net-(Q2-G): track 62.2 -> 61.7 mm
- added copper zone on B.Cu, net GND
- added copper zone on B.Cu, net GNDA
Other:
- outline, holes or cut-outs redrawn
- board text added: "FIX ground fills and find good connection point -sharp edges are issues?? -weird islands -large single enged connections -power planes -back layer (power or gnd??) -main cutoff switch -analog ground to adc -user input"
- board text removed: "FIX ground fills and find good connection point' -weird islands -large single enged connections -power planes -back layer (power or gnd??)"

Commit message: Its going
Parts:
- removed C13, C14, C20, C23: 1uF, Capacitor_SMD:C_0402_1005Metric_Pad0.74x0.62mm_HandSolder
- removed C15, C24: 10uF, Capacitor_SMD:C_0603_1608Metric_Pad1.08x0.95mm_HandSolder
- removed C17, C19, C21, C22, C28: 100nF, Capacitor_SMD:C_0402_1005Metric_Pad0.74x0.62mm_HandSolder
- removed D1: LED, LED_SMD:LED_0603_1608Metric_Pad1.05x0.95mm_HandSolder
- removed R1, R3, R57: 100K, Resistor_SMD:R_0603_1608Metric_Pad0.98x0.95mm_HandSolder
- removed R12: 1k, Resistor_SMD:R_0603_1608Metric_Pad0.98x0.95mm_HandSolder
- removed R13, R19, R27, R49: 1K, Resistor_SMD:R_0603_1608Metric_Pad0.98x0.95mm_HandSolder
- removed R14: 300K, Resistor_SMD:R_0402_1005Metric_Pad0.72x0.64mm_HandSolder
- removed R24, R70: 0R, Resistor_SMD:R_0603_1608Metric_Pad0.98x0.95mm_HandSolder
- removed R60: 1M, Resistor_SMD:R_0603_1608Metric_Pad0.98x0.95mm_HandSolder
- removed R64: 10K, Resistor_SMD:R_0603_1608Metric_Pad0.98x0.95mm_HandSolder
- removed R69: 145K, Resistor_SMD:R_0603_1608Metric_Pad0.98x0.95mm_HandSolder
- removed TP1, TP2, TP3, TP4: TestPoint, TestPoint:TestPoint_Pad_D2.0mm
- removed U12: XC62KN33302PR-G, Package_TO_SOT_SMD:SOT-89-3
- removed U13, U14, U16: CPC1017N, Package_SO:SOP-4_3.8x4.1mm_P2.54mm
- removed U2: LM358, Package_SO:SOP-8_3.9x4.9mm_P1.27mm
- added C27: 100nF, Capacitor_SMD:C_0402_1005Metric_Pad0.74x0.62mm_HandSolder, F.Cu at (114.9, 42.6)
- added C30: 100nF, Capacitor_SMD:C_0402_1005Metric_Pad0.74x0.62mm_HandSolder, F.Cu at (114.9, 44.6)
- added C35: 100nF, Capacitor_SMD:C_0402_1005Metric_Pad0.74x0.62mm_HandSolder, F.Cu at (114.9, 46.5)
- added C41: 1uF, Capacitor_SMD:C_0402_1005Metric_Pad0.74x0.62mm_HandSolder, F.Cu at (112.3, 78.2)
- added C42: 100nF, Capacitor_SMD:C_0402_1005Metric_Pad0.74x0.62mm_HandSolder, F.Cu at (112.3, 80.2)
- added C43: 100nF, Capacitor_SMD:C_0402_1005Metric_Pad0.74x0.62mm_HandSolder, F.Cu at (112.3, 82.2)
- added C44: 1uF, Capacitor_SMD:C_0402_1005Metric_Pad0.74x0.62mm_HandSolder, F.Cu at (112.3, 84.1)
- added D6: LED, LED_SMD:LED_0603_1608Metric_Pad1.05x0.95mm_HandSolder, F.Cu at (116.1, 78.5)
- added R73: 1K, Resistor_SMD:R_0603_1608Metric_Pad0.98x0.95mm_HandSolder, F.Cu at (98.0, 47.9)
- added R74: 1K, Resistor_SMD:R_0603_1608Metric_Pad0.98x0.95mm_HandSolder, F.Cu at (98.0, 50.4)
- added R75: 1K, Resistor_SMD:R_0603_1608Metric_Pad0.98x0.95mm_HandSolder, F.Cu at (98.0, 52.9)
- added SW2: SW_Push, Button_Switch_SMD:SW_SPST_B3S-1000, F.Cu at (107.8, 45.9)
- added SW3: SW_Push, Button_Switch_SMD:SW_SPST_B3S-1000, F.Cu at (107.8, 54.3)
- added SW4: SW_Push, Button_Switch_SMD:SW_SPST_B3S-1000, F.Cu at (107.8, 62.8)
- added U23: CPC1017N, Package_SO:SOP-4_3.8x4.1mm_P2.54mm, F.Cu at (91.6, 50.1)
- added U24: AMS1117-5.0, Package_TO_SOT_SMD:SOT-223-3_TabPin2, F.Cu at (115.6, 73.1)
- added U26: TL7660CDR, Package_SO:SOIC-8_3.9x4.9mm_P1.27mm, F.Cu at (106.5, 72.2)
- added U27: TL7660CDR, Package_SO:SOIC-8_3.9x4.9mm_P1.27mm, F.Cu at (106.5, 78.7)
- added U28: TL7660CDR, Package_SO:SOIC-8_3.9x4.9mm_P1.27mm, F.Cu at (106.5, 85.1)
- added U29: CPC1017N, Package_SO:SOP-4_3.8x4.1mm_P2.54mm, F.Cu at (91.6, 55.8)
- added U30: CPC1017N, Package_SO:SOP-4_3.8x4.1mm_P2.54mm, F.Cu at (91.6, 61.4)
- added U31: CPC1017N, Package_SO:SOP-4_3.8x4.1mm_P2.54mm, F.Cu at (91.6, 67.0)
- R54: value 10K -> 100K
- R63: value 0R -> 1K
- R66: value 10K -> 1K
- R67: value 10K -> 1k
- R68: value 300K -> 100R
- U22: value OPA2140 -> CPC1017N; footprint Package_SO:SOP-8_3.9x4.9mm_P1.27mm -> Package_SO:SOP-4_3.8x4.1mm_P2.54mm
- moved U22 85.2 mm to (91.6, 44.5), turned to 0 degrees
- moved R68 84.7 mm to (97.5, 55.2), turned to 0 degrees
- moved R66 82.3 mm to (98.0, 45.4), turned to 0 degrees
- moved R63 81.8 mm to (98.0, 42.9), turned to 0 degrees
- moved C25 76.3 mm to (97.5, 57.1), turned to 0 degrees
- moved R67 72.0 mm to (116.1, 81.1), turned to 0 degrees
Connections:
- net /Measurement Analog/100V renamed Net-(R54-Pad1)
- C11 pad 1: 3Vref -> +3.3V
- C12 pad 1: 3Vref -> +3.3V
- C16 pad 1: BattOut+ -> +9V
- C25 pad 1: +3.3V -> OpAmpIn
- C5 pad 1: BattOut+ -> +9V
- C6 pad 1: +3.3V -> OpAmpSupply+
- C7 pad 2: -3V3 -> OpAmpSupply-
- J8 pad 1: BattOut+ -> +9V
- J9 pad 1: BattOut- -> GND
- Q6 pad 2: 3Vref -> +3.3V
- R29 pad 1: InputPos -> Net-(U5A--)
- R29 pad 2: Net-(U5A-+) -> BufferOut
- R63 pad 1: CurrentOut -> GPIO_3
- R63 pad 2: Net-(U22A-+) -> Net-(R63-Pad2)
- R66 pad 1: Net-(U22A--) -> GPIO_4
- R66 pad 2: Net-(U22B-+) -> Net-(R66-Pad2)
- R67 pad 1: GNDA -> Net-(D6-K)
- R67 pad 2: Net-(U22B--) -> GND
- R68 pad 1: Net-(U22B-+) -> OpAmpIn
- R68 pad 2: 3Vref -> Net-(U5A-+)
- U22 pad 1: Net-(U22A--) -> Net-(R63-Pad2)
- U22 pad 2: Net-(U22A--) -> GND
- U22 pad 3: Net-(U22A-+) -> OpAmpIn
- U22 pad 4: -3V3 -> InputPos
- U5 pad 4: -3V3 -> OpAmpSupply-
- U5 pad 8: +3.3V -> OpAmpSupply+
- U7 pad 2: unconnected-(U7-PC13-Pad2) -> VButton
- U7 pad 3: unconnected-(U7-PC14-Pad3) -> CButton
- U7 pad 39: unconnected-(U7-PB3-Pad39) -> GPIO_17
- U7 pad 4: unconnected-(U7-PC15-Pad4) -> RButton
- U7 pad 41: unconnected-(U7-PB5-Pad41) -> GPIO_16
- U8 pad 3: BattOut+ -> +9V
Routing:
- net (no net): track 0.00 -> 78.8 mm, vias 0 -> 2
- net GND: track 5.63 -> 34.9 mm
- net BattOut-: track 29.2 -> 0.00 mm
- net Net-(U22A-+): track 18.8 -> 0.00 mm, vias 2 -> 0
- net -3V3: track 12.0 -> 0.00 mm
- net Net-(U22A--): track 7.94 -> 0.00 mm
- net /Measurement Analog/1000V: track 4.76 -> 0.00 mm
- net Net-(R69-Pad2): track 4.44 -> 0.00 mm
- net /Measurement Analog/1V: track 4.35 -> 0.00 mm
- net /Measurement Analog/10V: track 4.20 -> 0.00 mm
- net Net-(U2A-+): track 3.97 -> 0.00 mm
- net Net-(U22B--): track 3.84 -> 0.00 mm
- net Net-(U22B-+): track 3.39 -> 0.00 mm
- net Net-(U2A--): track 3.15 -> 0.00 mm
- net 3Vref: track 4.37 -> 1.38 mm
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