File: HandHeldDMM-main/DMMVoltageRanges.kicad_sch (KiCad schematic)
At the start: 97 parts, among them Q1 HD6362, Q10 SI2301, Q11 SI2301, Q12 SI2301, Q2 HD6362, Q3 SI2302, Q4 SI2302, Q5 SI2302, Q6 SI2301, Q7 SI2301, Q8 HD6362, Q9 SI2301, U1 TLP291, U10 TLP291, U11 LM334M, U13 CPC1017N, U14 CPC1017N, U15 CPC1017N, U16 CPC1017N, U17 TLP291, U18 TLP291, U19 TLP291, U20 TLP291, U21 TLP291, U22 OPA2140, U3 TLP291, U4 TLP291, U5 OPA2140, U6 TLP291, U9 TLP291

Commit message: More pcb work
Parts:
- R28, R29, R63, R70: footprint Resistor_SMD:R_0402_1005Metric_Pad0.72x0.64mm_HandSolder -> Resistor_SMD:R_0603_1608Metric_Pad0.98x0.95mm_HandSolder; LCSC Price 0.05 -> 0.09; Store https://www.lcsc.com/product-detail/Chip-Resistor-Surface-Mount_FOJAN-FRC0402P000-TS_C2906877.html -> https://www.lcsc.com/product-detail/Chip-Resistor-Surface-Mount_FOJAN-FRC0603P000-TS_C2907080.html
Changed lines of the file:
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@@
       (effects (font (size 1.27 1.27)))
     )
-    (property "Footprint" "Resistor_SMD:R_0402_1005Metric_Pad0.72x0.64mm_HandSolder" (at 221.615 58.928 90)
-      (effects (font (size 1.27 1.27)) hide)
-    )
-    (property "Datasheet" "https://datasheet.lcsc.com/lcsc/2308241947_FOJAN-FRC0402P000-TS_C2906877.pdf" (at 221.615 57.15 0)
-      (effects (font (size 1.27 1.27)) hide)
-    )
-    (property "Store" "https://www.lcsc.com/product-detail/Chip-Resistor-Surface-Mount_FOJAN-FRC0402P000-TS_C2906877.html" (at 221.615 57.15 90)
-      (effects (font (size 1.27 1.27)) hide)
-    )
-    (property "LCSC Price" "0.05" (at 221.615 57.15 0)
+    (property "Footprint" "Resistor_SMD:R_0603_1608Metric_Pad0.98x0.95mm_HandSolder" (at 221.615 58.928 90)
+      (effects (font (size 1.27 1.27)) hide)
+    )
+    (property "Datasheet" "https://datasheet.lcsc.com/lcsc/2308241947_FOJAN-FRC0603P000-TS_C2907080.pdf" (at 221.615 57.15 0)
+      (effects (font (size 1.27 1.27)) hide)
+    )
+    (property "Store" "https://www.lcsc.com/product-detail/Chip-Resistor-Surface-Mount_FOJAN-FRC0603P000-TS_C2907080.html" (at 221.615 57.15 90)
+      (effects (font (size 1.27 1.27)) hide)
+    )
+    (property "LCSC Price" "0.09" (at 221.615 57.15 0)
       (effects (font (size 1.27 1.27)) hide)
     )
@@
       (effects (font (size 1.27 1.27)))
     )
-    (property "Footprint" "Resistor_SMD:R_0402_1005Metric_Pad0.72x0.64mm_HandSolder" (at 322.58 211.328 90)
-      (effects (font (size 1.27 1.27)) hide)
-    )
-    (property "Datasheet" "https://datasheet.lcsc.com/lcsc/2308241947_FOJAN-FRC0402P000-TS_C2906877.pdf" (at 322.58 209.55 0)
-      (effects (font (size 1.27 1.27)) hide)
-    )
-    (property "LCSC Price" "0.05" (at 322.58 209.55 0)
+    (property "Footprint" "Resistor_SMD:R_0603_1608Metric_Pad0.98x0.95mm_HandSolder" (at 322.58 211.328 90)
+      (effects (font (size 1.27 1.27)) hide)
+    )
+    (property "Datasheet" "https://datasheet.lcsc.com/lcsc/2308241947_FOJAN-FRC0603P000-TS_C2907080.pdf" (at 322.58 209.55 0)
+      (effects (font (size 1.27 1.27)) hide)
+    )
+    (property "LCSC Price" "0.09" (at 322.58 209.55 0)
       (effects (font (size 1.27 1.27)) hide)
     )
@@
       (effects (font (size 1.27 1.27)) hide)
     )
-    (property "Store" "https://www.lcsc.com/product-detail/Chip-Resistor-Surface-Mount_FOJAN-FRC0402P000-TS_C2906877.html" (at 322.58 209.55 0)
+    (property "Store" "https://www.lcsc.com/product-detail/Chip-Resistor-Surface-Mount_FOJAN-FRC0603P000-TS_C2907080.html" (at 322.58 209.55 0)
       (effects (font (size 1.27 1.27)) hide)
     )
@@
       (effects (font (size 1.27 1.27)))
     )
-    (property "Footprint" "Resistor_SMD:R_0402_1005Metric_Pad0.72x0.64mm_HandSolder" (at 309.245 64.008 90)
-      (effects (font (size 1.27 1.27)) hide)
-    )
-    (property "Datasheet" "https://datasheet.lcsc.com/lcsc/2308241947_FOJAN-FRC0402P000-TS_C2906877.pdf" (at 309.245 62.23 0)
-      (effects (font (size 1.27 1.27)) hide)
-    )
-    (property "LCSC Price" "0.05" (at 309.245 62.23 0)
+    (property "Footprint" "Resistor_SMD:R_0603_1608Metric_Pad0.98x0.95mm_HandSolder" (at 309.245 64.008 90)
+      (effects (font (size 1.27 1.27)) hide)
+    )
+    (property "Datasheet" "https://datasheet.lcsc.com/lcsc/2308241947_FOJAN-FRC0603P000-TS_C2907080.pdf" (at 309.245 62.23 0)
+      (effects (font (size 1.27 1.27)) hide)
+    )
+    (property "LCSC Price" "0.09" (at 309.245 62.23 0)
       (effects (font (size 1.27 1.27)) hide)
     )
@@
       (effects (font (size 1.27 1.27)) hide)
     )
-    (property "Store" "https://www.lcsc.com/product-detail/Chip-Resistor-Surface-Mount_FOJAN-FRC0402P000-TS_C2906877.html" (at 309.245 62.23 0)
+    (property "Store" "https://www.lcsc.com/product-detail/Chip-Resistor-Surface-Mount_FOJAN-FRC0603P000-TS_C2907080.html" (at 309.245 62.23 0)
       (effects (font (size 1.27 1.27)) hide)
     )
@@
       (effects (font (size 1.27 1.27)))
     )
-    (property "Footprint" "Resistor_SMD:R_0402_1005Metric_Pad0.72x0.64mm_HandSolder" (at 237.49 206.248 90)
-      (effects (font (size 1.27 1.27)) hide)
-    )
-    (property "Datasheet" "https://datasheet.lcsc.com/lcsc/2308241947_FOJAN-FRC0402P000-TS_C2906877.pdf" (at 237.49 204.47 0)
-      (effects (font (size 1.27 1.27)) hide)
-    )
-    (property "Store" "https://www.lcsc.com/product-detail/Chip-Resistor-Surface-Mount_FOJAN-FRC0402P000-TS_C2906877.html" (at 237.49 204.47 90)
-      (effects (font (size 1.27 1.27)) hide)
-    )
-    (property "LCSC Price" "0.05" (at 237.49 204.47 0)
-      (effects (font (size 1.27 1.27)) hide)
-    )
+    (property "Footprint" "Resistor_SMD:R_0603_1608Metric_Pad0.98x0.95mm_HandSolder" (at 237.49 206.248 90)
+      (effects (font (size 1.27 1.27)) hide)
+    )
+    (property "Datasheet" "https://datasheet.lcsc.com/lcsc/2308241947_FOJAN-FRC0603P000-TS_C2907080.pdf" (at 237.49 204.47 0)
+      (effects (font (size 1.27 1.27)) hide)
+    )
+    (property "Store" "https://www.lcsc.com/product-detail/Chip-Resistor-Surface-Mount_FOJAN-FRC0603P000-TS_C2907080.html" (at 237.49 204.47 90)
+      (effects (font (size 1.27 1.27)) hide)
+    )
+    (property "LCSC Price" "0.09" (at 237.49 204.47 0)
+      (effects (font (size 1.27 1.27)) hide)
+    )

Commit message: PCB rev 1 with schematic change ideas
Other:
- note added: "Both use the top opamps"
- note added: "Op-amp capacitor / resistor - smooth input - prevent 140 from dying"
- note added: "Parallel resiters can improve ppm specs"
- note added: "Shifting voltages down then back up is prone to lots of noise"
- note added: "dont need percision 3v ref - buffer from ref source for current"
- note added: "problems with low voltage and accurate measurements ofver resisters"
Changed lines of the file:
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@@
+    (effects (font (size 1.27 1.27)) (justify left bottom))
+  )
+  (text "Op-amp capacitor / resistor\n- smooth input\n- prevent 140 from dying"
+    (at 213.36 30.48 0)
     (effects (font (size 1.27 1.27)) (justify left bottom))
   )
@@
     (effects (font (size 2 2) (thickness 0.4) bold) (justify left bottom))
   )
+  (text "Shifting voltages down then back up is prone to lots of noise"
+    (at 287.02 27.94 0)
+    (effects (font (size 1.27 1.27)) (justify left bottom))
+  )
+  (text "Parallel resiters can improve ppm specs" (at 255.905 375.285 0)
+    (effects (font (size 1.27 1.27)) (justify left bottom))
+  )
+  (text "dont need percision 3v ref\n- buffer from ref source for current"
+    (at 55.88 292.735 0)
+    (effects (font (size 1.27 1.27)) (justify left bottom))
+  )
   (text "ADC Input Conditioning" (at 247.65 38.1 0)
     (effects (font (size 2 2) (thickness 0.4) bold) (justify left bottom))
@@
     (effects (font (size 1.27 1.27)) (justify left bottom))
   )
+  (text "Both use the top opamps" (at 261.62 170.18 0)
+    (effects (font (size 1.27 1.27)) (justify left bottom))
+  )
   (text "10A" (at 66.04 241.3 0)
     (effects (font (size 1.27 1.27)) (justify left bottom))
@@
     (effects (font (size 1.27 1.27)) (justify left bottom))
   )
+  (text "problems with low voltage and accurate measurements ofver resisters"
+    (at 57.785 35.56 0)
+    (effects (font (size 1.27 1.27)) (justify left bottom))
+  )

Commit message: Its going
Parts:
- removed C28: 100nF, Capacitor_SMD:C_0402_1005Metric_Pad0.74x0.62mm_HandSolder, symbol Device:C
- removed R13, R19, R27, R49: 1K, Resistor_SMD:R_0603_1608Metric_Pad0.98x0.95mm_HandSolder, symbol Device:R
- removed R14: 300K, Resistor_SMD:R_0402_1005Metric_Pad0.72x0.64mm_HandSolder, symbol Device:R
- removed R57: 100K, Resistor_SMD:R_0603_1608Metric_Pad0.98x0.95mm_HandSolder, symbol Device:R
- removed R60: 1M, Resistor_SMD:R_0603_1608Metric_Pad0.98x0.95mm_HandSolder, symbol Device:R
- removed R64, R67: 10K, Resistor_SMD:R_0603_1608Metric_Pad0.98x0.95mm_HandSolder, symbol Device:R
- removed U13, U14, U16: CPC1017N, Package_SO:SOP-4_3.8x4.1mm_P2.54mm, symbol Relay_SolidState:CPC1017N
- removed U22: OPA2140, Package_SO:SOP-8_3.9x4.9mm_P1.27mm, symbol Amplifier_Operational:OPA2134
- added R73, R74, R75: 1K, Resistor_SMD:R_0603_1608Metric_Pad0.98x0.95mm_HandSolder, symbol Device:R
- added U22, U23, U29, U30, U31: CPC1017N, Package_SO:SOP-4_3.8x4.1mm_P2.54mm, symbol Relay_SolidState:CPC1017N
- R54: value 10K -> 100K
- R63: value 0R -> 1K; LCSC Price 0.09 -> copy; Price Qty 100 -> copy; Store https://www.lcsc.com/product-detail/Chip-Resistor-Surface-M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 -> https://www.lcsc.com/product-detail/Chip-span-style-backgro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
- R66: value 10K -> 1K; LCSC Price 0.1 -> copy; Price Qty 100 -> copy; Store https://www.lcsc.com/product-detail/Chip-Resistor-Surface-M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 -> https://www.lcsc.com/product-detail/Chip-span-style-backgro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
- R68: value 300K -> 100R; LCSC Price 0.06 -> 0.05; Store https://www.lcsc.com/product-detail/Chip-Resistor-Surface-M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 -> https://www.lcsc.com/product-detail/Chip-span-style-backgro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
- R69: value 145K -> 4K; footprint Resistor_SMD:R_0603_1608Metric_Pad0.98x0.95mm_HandSolder -> (none); LCSC Price 0.7 -> (none); Price Qty 10 -> (none); Store https://www.lcsc.com/product-detail/Chip-Resistor-Surface-M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 -> (none)
- R70: value 0R -> 1K; footprint Resistor_SMD:R_0603_1608Metric_Pad0.98x0.95mm_HandSolder -> (none); LCSC Price 0.09 -> (none); Price Qty 100 -> (none); Store https://www.lcsc.com/product-detail/Chip-Resistor-Surface-M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 -> (none)
Connections:
- net SD-ADC2 is gone; now on net SD-ADC1: R70.2
- net +3.3V: now also C11.1, C12.1, Q6.2 (S); no longer C25.1, C6.1, U5.8 (V+)
- net CurrentOut: now also U23.3; no longer R63.1
- net GND: now also U22.2, U23.2, U29.2, U30.2, U31.2
- net GNDA: now also R70.1
- net GPIO_3: now also R63.1
- net GPIO_4: now also R66.1, R74.1, R75.1
- net GPIO_5: now also R73.1
- net InputPos: now also U22.4; no longer R29.1
- net SD-ADC1: now also R69.2, U29.3
- net at U5.3 (+): now also R68.2; no longer R29.2
- net at U5.1, U5.2 (-): now also R29.1
- net at U5.5 (+): now also U31.3
- net at R66.2: now also U23.1; no longer R68.1
- net at R69.1: now also U30.3
- net at R63.2: now also U22.1
- net -3V3 renamed OpAmpSupply-
- net 100V: no longer names the net of R54.1, U15.3
- removed net 3Vref: C11.1, C12.1, Q6.2 (S), R68.2
- new net: R75.2, U31.1
- new net: R74.2, U30.1
- new net: R73.2, U29.1
- new net BufferOut: R29.2, U29.4, U30.4, U31.4
- new net OpAmpIn: C25.1, R68.1, U22.3, U23.4
- new net OpAmpSupply+: C6.1, U5.8 (V+)
Other:
- note added: "10v out max"
- note added: "200V"
- note added: "Equations: Current Value R-Set Value Ohms Range LCSC 0.064 = 0.000001A * R; Amps = 1uA R = 64,000 ohms 100k - 1M https://www.lcsc.com/product-detail/Chip-span-style-background-color-ff0-Resistor-span-Surface-Mount_Viking-Tech-ARG03DTC6402N_C2902643.html 0.064 = 0.000002A * R; Amps = 2uA R = 32,000 ohms 0.064 = 0.000005A * R; Amps = 5uA R = 12,800 ohms 0.064 = 0.00800A * R; Amps = 8uA R = 8,000 oh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"
- note added: "Have to live with low voltage out from current in order to minimize burden voltage on DUT that could change measurement"
- note added: "Make ranges 2's 200mV 2V 10V (maybe 15V) 200V Straight in for 100mV - 10V 200V range scaled down to 10V for buffer then 2V for adc scaled to 2v for adc 2V scaled allows there to be overshoot on each range, not a hard cap at 2V"
- note added: "OPAMP CMV common mode voltage adds context to rail to rail supply!!"
- note added: "what value??"
- note removed: "Bipolar to unipolar converter Output range = 0-3v"
- note removed: "Both use the top opamps"
- moved on the sheet: C6, C7, R15, R16, R2, R25, R28, R29, R54, U15, U5A, U5B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

Commit message: Layout / routing V2 with schematic fixes
Parts:
- removed C11: 100nF, Capacitor_SMD:C_0402_1005Metric_Pad0.74x0.62mm_HandSolder, symbol Device:C
- removed C12: 1uF, Capacitor_SMD:C_0402_1005Metric_Pad0.74x0.62mm_HandSolder, symbol Device:C
- added R1: 1K, Resistor_SMD:R_0603_1608Metric_Pad0.98x0.95mm_HandSolder, symbol Device:R
- C25, C6, C7: LCSC Price 0 -> 0.18; PART# (none) -> C513772; Price / 1 (none) -> 0.0018; Price Qty 0 -> 100; Store Parts Bin -> https://www.lcsc.com/product-detail/Multilayer-Ceramic-Capa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
- Q1, Q2, Q8: PART# (none) -> C5451644; Price / 1 (none) -> 0.2124
- Q10, Q11, Q12, Q6, Q7, Q9: PART# (none) -> C5261052; Price / 1 (none) -> 0.0117
- Q3, Q4, Q5: PART# (none) -> C4748714; Price / 1 (none) -> 0.0116
- R11, R4, R5, R52, R55, R58, R6, R61, R62, R68, R7, R8: PART# (none) -> C2906860; Price / 1 (none) -> 0.0005
- R15: value 10K -> 1K; LCSC Price 0.1 -> 0.25; PART# (none) -> C5141145; Price / 1 (none) -> 0.0049; Price Qty 100 -> 50; Store https://www.lcsc.com/product-detail/Chip-Resistor-Surface-M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 -> https://www.lcsc.com/product-detail/Chip-span-style-backgro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
- R16: value 145K -> 18K; footprint Resistor_SMD:R_0603_1608Metric_Pad0.98x0.95mm_HandSolder -> Resistor_SMD:R_0402_1005Metric_Pad0.72x0.64mm_HandSolder; LCSC Price 0.7 -> 0.45; PART# (none) -> C2984412; Price / 1 (none) -> 0.0224; Price Qty 10 -> 20; Store https://www.lcsc.com/product-detail/Chip-Resistor-Surface-M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 -> https://www.lcsc.com/product-detail/Chip-span-style-backgro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
- R17: PART# (none) -> C105063; Price / 1 (none) -> 0.0185
- R18: PART# (none) -> C5127856; Price / 1 (none) -> 0.0886
- R2, R21, R31, R33, R34, R35, R50, R51, R53, R56, R59: PART# (none) -> C2906980; Price / 1 (none) -> 0.0009
- R20: PART# (none) -> C508576; Price / 1 (none) -> 0.2564
- R22: PART# (none) -> C841792; Price / 1 (none) -> 0.0761
- R23: PART# (none) -> C105071; Price / 1 (none) -> 0.0242
- R25, R63, R66, R73, R74, R75: LCSC Price copy -> 0.25; PART# (none) -> C5141145; Price / 1 (none) -> 0.0049; Price Qty copy -> 50
- R28, R29: PART# (none) -> C2907080; Price / 1 (none) -> 0.0009
- R32: PART# (none) -> C3014413; Price / 1 (none) -> 0.0083
- R37, R41, R42, R43: PART# (none) -> C2933075; Price / 1 (none) -> 0.0005
- R38, R40, R45, R47: PART# (none) -> C3015729; Price / 1 (none) -> 0.0005
- R39, R44, R46, R48: PART# (none) -> C3015705; Price / 1 (none) -> 0.0007
- R54: LCSC Price 0.1 -> 0.09; PART# (none) -> C2906980; Price / 1 (none) -> 0.0009; Store https://www.lcsc.com/product-detail/Chip-Resistor-Surface-Mount_RALEC-RTT031002FTP_C103199.html -> https://www.lcsc.com/product-detail/Chip-Resistor-Surface-Mount_FOJAN-FRC0603F1003TS_C2906980.html
- R65: PART# (none) -> C3037190; Price / 1 (none) -> 0.0037
- R69: footprint (none) -> Resistor_SMD:R_0603_1608Metric_Pad0.98x0.95mm_HandSolder; LCSC Price (none) -> 0.42; PART# (none) -> C2984443; Price / 1 (none) -> 0.0083; Price Qty (none) -> 50; Store (none) -> https://www.lcsc.com/product-detail/Chip-Resistor-Surface-M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
- R70: footprint (none) -> Resistor_SMD:R_0603_1608Metric_Pad0.98x0.95mm_HandSolder; LCSC Price (none) -> 0.25; PART# (none) -> C5141145; Price / 1 (none) -> 0.0049; Price Qty (none) -> 50; Store (none) -> https://www.lcsc.com/product-detail/Chip-span-style-backgro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
- U1, U10, U17, U18, U19, U20, U21, U3, U4, U6, U9: PART# (none) -> C3018819; Price / 1 (none) -> 0.0882
- U11: PART# (none) -> C7945; Price / 1 (none) -> 0.655
- U15, U22, U23, U29, U30, U31: PART# (none) -> C81521; Price / 1 (none) -> 0.67
- U5: PART# (none) -> C335586; Price / 1 (none) -> 3.8278
Connections:
- net BufferOut: now also U30.3; no longer U30.4
- net CurrentOut: now also U23.4; no longer U23.3
- net GNDA: now also R1.1; no longer R15.1
- net InputPos: now also U15.3, U22.3; no longer U15.4, U22.4
- net OpAmpIn: now also U22.4, U23.3; no longer U22.3, U23.4
- net at R69.1: now also U30.4; no longer U30.3
- net at R54.1: now also U15.4; no longer U15.3
- net GPIO_10 renamed OOpto1
- net GPIO_11 renamed OOpto2
- net GPIO_12 renamed OOpto3
- net GPIO_13 renamed OOpto4
- net GPIO_14 renamed OOpto5
- net GPIO_15 renamed OOpto6
- net GPIO_2 renamed VOpto1
- net GPIO_3 renamed ADCOpto2
- removed net GPIO_4: R66.1, R74.1, R75.1
- net GPIO_5 renamed ADCOpto3
- net ADCOpto3: no longer R4.1
- net GPIO_6 renamed AOpto2
- net GPIO_7 renamed AOpto3
- net GPIO_8 renamed AOpto4
- net GPIO_9 renamed AOpto5
- new net: R1.2, R15.1
- new net ADCOpto1: R66.1
- new net ADCOpto4: R74.1
- new net ADCOpto5: R75.1
- new net AOpto1: R4.1
Other:
- note added: "Great Resistor calculator https://jansson.us/resistors.html"
- note added: "Rf"
- note added: "Rin"
- moved on the sheet: R54, R66, R69, R70, U23

Commit message: Finished?
Other:
- moved on the sheet: C6, C7, R63, R66, U22, U23, U5C

Commit message: Ordered
Parts:
- R20: LCSC Price 0.93 -> 1.62; PART# C508576 -> C487937; Price / 1 0.2564 -> 0.404; Store https://www.lcsc.com/product-detail/Current-Sense-Resistors-span-style-background-color-ff0-Shunt-span-Resistors_Milliohm-HoLR-5W-10mR-1-JZ-10_C508576.html -> https://www.lcsc.com/product-detail/Current-Sense-Resistors-Shunt-Resistors_Shenzhen-Yezhan-Elec-J5-10-10F-t-y_C487937.html
Changed lines of the file:
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@@
       (effects (font (size 1.27 1.27)) hide)
     )
-    (property "Datasheet" "https://datasheet.lcsc.com/lcsc/2004112132_Milliohm-HoLR-5W-10mR-1--JZ-10_C508576.pdf" (at 56.515 241.3 0)
+    (property "Datasheet" "https://datasheet.lcsc.com/lcsc/2310300938_Shenzhen-Yezhan-Elec--J5-10-10F-t-y_C487937.pdf" (at 56.515 241.3 0)
       (effects (font (size 1.27 1.27)) hide)
     )
-    (property "Store" "https://www.lcsc.com/product-detail/Current-Sense-Resistors-span-style-background-color-ff0-Shunt-span-Resistors_Milliohm-HoLR-5W-10mR-1-JZ-10_C508576.html" (at 56.515 241.3 90)
+    (property "Store" "https://www.lcsc.com/product-detail/Current-Sense-Resistors-Shunt-Resistors_Shenzhen-Yezhan-Elec-J5-10-10F-t-y_C487937.html" (at 56.515 241.3 90)
       (effects (font (size 1.27 1.27)) hide)
     )
-    (property "LCSC Price" "0.93" (at 56.515 241.3 0)
+    (property "LCSC Price" "1.62" (at 56.515 241.3 0)
       (effects (font (size 1.27 1.27)) hide)
     )
@@
       (effects (font (size 1.27 1.27)) hide)
     )
-    (property "PART#" "C508576" (at 56.515 241.3 0)
+    (property "PART#" "C487937" (at 56.515 241.3 0)
       (effects (font (size 1.27 1.27)) hide)
     )
-    (property "Price / 1" "0.2564" (at 56.515 241.3 0)
+    (property "Price / 1" "0.404" (at 56.515 241.3 0)
       (effects (font (size 1.27 1.27)) hide)
     )

Commit message: schematic fixes
Parts:
- added D5, D6: 1N4007, Diode_THT:D_DO-41_SOD81_P10.16mm_Horizontal, symbol Diode:1N4007
Connections:
- net GND: now also D5.1 (K)
- net SD-ADC1: now also D5.2 (A), D6.2 (A)
- new net +3V3: D6.1 (K)
Other:
- note added: "200mV input (200mV range and 200V range) 2V out"
- note added: "20V max input 2V out"
- note added: "2V max"
- note added: "Values need to be 40 and 10K to prevent loading on the opamp (20mA max out)"
- note added: "need voltage on opamp to prevent from railing"
- note removed: "Layout Tips: - keep analog and digital grounds very well isolated!! - optocuplers are your friends"
- moved on the sheet: C25, C6, C7, Q1, Q10, Q11, Q12, Q2, Q3, Q4, Q5, Q6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
