File: HandHeldDMM-main/DMMVoltageRanges.kicad_sch (KiCad schematic)
At the start: 92 parts, among them Q1 HD6362, Q10 SI2301, Q11 SI2301, Q12 SI2301, Q2 HD6362, Q3 SI2302, Q4 SI2302, Q5 SI2302, Q6 SI2301, Q7 SI2301, Q8 HD6362, Q9 SI2301, U1 TLP291, U10 TLP291, U11 LM334M, U15 CPC1017N, U17 TLP291, U18 TLP291, U19 TLP291, U20 TLP291, U21 TLP291, U22 CPC1017N, U23 CPC1017N, U29 CPC1017N, U3 TLP291, U30 CPC1017N, U31 CPC1017N, U4 TLP291, U5 OPA2140, U6 TLP291, U9 TLP291

Commit message: fixes for v2
Connections:
- net GND: now also D5.2 (A); no longer D5.1 (K)
- net SD-ADC1: now also D5.1 (K); no longer D5.2 (A)
Other:
- note added: "10V max input 2V out"
- note added: "KILL- loads input circuit"
- note added: "Values need to be 40k and 10K to prevent loading on the opamp (2V max out 10V max in)(5:1)"
- note added: "add input resistance add 10K to ground to prevent floating inputs"
- note added: "add opto output control"
- note removed: "20V max input 2V out"
- note removed: "Values need to be 40 and 10K to prevent loading on the opamp (20mA max out)"
- note removed: "what value??"
- moved on the sheet: D5
Changed lines of the file:
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@@
     (effects (font (size 1.27 1.27)) (justify left bottom))
   )
-  (text "Values need to be 40 and 10K to prevent loading on the opamp\n(20mA max out)"
+  (text "Values need to be 40k and 10K to prevent loading on the opamp\n(2V max out 10V max in)(5:1)"
     (at 458.47 270.51 0)
     (effects (font (size 1.27 1.27)) (justify left bottom))
   )
+  (text "add input resistance\nadd 10K to ground to prevent floating inputs"
+    (at 508.635 313.055 0)
+    (effects (font (size 1.27 1.27)) (justify left bottom))
+  )
   (text "1mA" (at 178.435 196.215 0)
     (effects (font (size 1.27 1.27)) (justify left bottom))
@@
     (effects (font (size 1.27 1.27)) (justify left bottom))
   )
+  (text "add opto output control\n" (at 57.785 302.895 0)
+    (effects (font (size 1.27 1.27)) (justify left bottom))
+  )
   (text "\nEquations:             Current Value     R-Set Value        Ohms Range      LCSC\n0.064 = 0.000001A * R;  Amps = 1uA       R = 64,000 ohms    100k - 1M       https://www.lcsc.com/product-detail/Chip-span-style-background-color-ff0-Resistor-span-Surface-Mount_Viking-Tech-ARG03DTC6402N_C2902643.html\n0.064 = 0.000002A * R;  Amps = 2uA       R = 32,000 ohms    \n0.064 = 0.000005A * R;  Amps = 5uA       R = 12,800 ohms    \n0.064 = 0.00800A * R;   Amps = 8uA       R = 8,000 ohms     \n\n0.064 = 0.00001A * R;   Amps = 10uA      R = 6,400 ohms     10K - 100k      https://www.lcsc.com/product-detail/Chip-span-style-background-color-ff0-Resistor-span-Surface-Mount_Viking-Tech-ARG03DTC6401N_C3014413.html\n0.064 = 0.00002A * R;   Amps = 20uA      R = 3,200 ohms\n0.064 = 0.00005A * R;   Amps = 50uA      R = 1,280 ohms \n0.064 = 0.0080A * R;    Amps = 80uA      R = 800 ohms\n\n0.064 = 0.0001A * R;    Amps = 100uA     R = 640 ohms       1k - 10K        4 * (160) https://www.lcsc.com/product-detail/Chip-span-style-background-color-ff0-Resistor-span-Surface-Mount_Viking-Tech-ARG03DTC1600_C2758273.html\n0.064 = 0.0002A * R;    Amps = 200mA     R = 320 ohms\n0.064 = 0.0005A * R;    Amps = 500uA     R = 128 ohms \n0.064 = 0.008A * R;     Amps = 800uA     R = 80 ohms  \n   \n0.064 = 0.001A * R;     Amps = 1mA       R = 64 ohms        100 - 1k        4 * (16) https://www.lcsc.com/product-detail/Chip-Resistor-Surface-Mount_FOJAN-FRC0603F16R0TS_C2906998.html\n0.064 = 0.002A * R;     Amps = 2mA       R = 32 ohms\n0.064 = 0.005A * R;     Amps = 5mA       R = 12.8 ohms\n0.064 = 0.008A * R;     Amps = 8mA       R = 8 ohms\n\n0.064 = 0.01A * R;      Amps = 10mA      R = 6.4 ohms       10 - 100        4 * (1.6) https://www.lcsc.com/product-detail/Chip-Resistor-Surface-Mount_VO-SCR0603F1R6_C3016190.html\n"
     (at 287.02 149.225 0)
@@
     (effects (font (size 1.27 1.27)) (justify left bottom))
   )
-  (text "what value??" (at 340.36 260.35 0)
+  (text "KILL- loads input circuit" (at 337.185 260.35 0)
     (effects (font (size 1.27 1.27)) (justify left bottom))
   )
-  (text "20V max input\n2V out\n" (at 513.715 281.305 0)
+  (text "10V max input\n2V out\n" (at 513.715 281.305 0)
     (effects (font (size 1.27 1.27)) (justify left bottom))
   )
@@
   )
   (symbol (lib_id "Relay_SolidState:CPC1017N") (at 448.31 295.275 0) (unit 1)
-    (in_bom yes) (on_board yes) (dnp no) (fields_autoplaced)
+    (in_bom yes) (on_board yes) (dnp no)
     (property "Reference" "U31" (at 448.31 287.02 0)
       (effects (font (size 1.27 1.27)))
@@
     )
   )
-  (symbol (lib_id "Diode:1N4007") (at 540.385 194.31 90) (unit 1)
+  (symbol (lib_id "Diode:1N4007") (at 540.385 194.31 270) (unit 1)
     (in_bom yes) (on_board yes) (dnp no) (fields_autoplaced)
-    (property "Reference" "D5" (at 542.925 193.04 90)
-      (effects (font (size 1.27 1.27)) (justify right))
+    (property "Reference" "D5" (at 543.56 193.04 90)
+      (effects (font (size 1.27 1.27)) (justify left))
     )
-    (property "Value" "1N4007" (at 542.925 195.58 90)
-      (effects (font (size 1.27 1.27)) (justify right))
+    (property "Value" "1N4007" (at 543.56 195.58 90)
+      (effects (font (size 1.27 1.27)) (justify left))
     )
-    (property "Footprint" "Diode_THT:D_DO-41_SOD81_P10.16mm_Horizontal" (at 544.83 194.31 0)
+    (property "Footprint" "Diode_THT:D_DO-41_SOD81_P10.16mm_Horizontal" (at 535.94 194.31 0)
       (effects (font (size 1.27 1.27)) hide)
     )
