File: HandHeldDMM-main/DMMVoltageRanges.kicad_sch (KiCad schematic)
At the start: 92 parts, among them Q1 HD6362, Q10 SI2301, Q11 SI2301, Q12 SI2301, Q2 HD6362, Q3 SI2302, Q4 SI2302, Q5 SI2302, Q6 SI2301, Q7 SI2301, Q8 HD6362, Q9 SI2301, U1 TLP291, U10 TLP291, U11 LM334M, U15 CPC1017N, U17 TLP291, U18 TLP291, U19 TLP291, U20 TLP291, U21 TLP291, U22 CPC1017N, U23 CPC1017N, U29 CPC1017N, U3 TLP291, U30 CPC1017N, U31 CPC1017N, U4 TLP291, U5 OPA2140, U6 TLP291, U9 TLP291

Commit message: schematic changes
Other:
- note added: "10V range 2V out"
- note added: "200mV range 2V out"
- note added: "2V and 200V (scaled to 2V) ranges"
- note added: "2V out max"
- note added: "Make ranges 2's 200mV 2V 10V (maybe 15V) 200V Straight in for 2V range and 200V range (scaled to 2V) 200V range scaled down to 2V 2V scaled allows there to be overshoot on each range, not a hard cap at 2V"
- note removed: "10V max input 2V out"
- note removed: "10v out max"
- note removed: "200mV input (200mV range and 200V range) 2V out"
- note removed: "2V max"
- note removed: "Make ranges 2's 200mV 2V 10V (maybe 15V) 200V Straight in for 100mV - 10V 200V range scaled down to 10V for buffer then 2V for adc scaled to 2v for adc 2V scaled allows there to be overshoot on each range, not a hard cap at 2V"
Changed lines of the file:
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@@
     (effects (font (size 2 2) (thickness 0.4) bold) (justify left bottom))
   )
-  (text "2V max" (at 485.775 257.81 0)
+  (text "2V and 200V (scaled to 2V) ranges" (at 475.488 257.302 0)
     (effects (font (size 1.27 1.27)) (justify left bottom))
   )
@@
     (effects (font (size 1.27 1.27)) (justify left bottom))
   )
-  (text "10v out max" (at 113.665 98.425 0)
+  (text "2V out max" (at 114.808 98.552 0)
     (effects (font (size 1.27 1.27)) (justify left bottom))
   )
@@
     (effects (font (size 1.27 1.27)) (justify left bottom))
   )
-  (text "200mV input (200mV range and 200V range)\n2V out" (at 503.555 294.64 0)
+  (text "200mV range\n2V out" (at 502.412 297.434 0)
     (effects (font (size 1.27 1.27)) (justify left bottom))
   )
-  (text "Make ranges 2's 200mV 2V 10V (maybe 15V) 200V\n\nStraight in for 100mV - 10V \n\n200V range scaled down to 10V for buffer then 2V for adc\n\n\nscaled to 2v for adc\n2V scaled allows there to be overshoot on each range, not a hard cap at 2V\n"
+  (text "Make ranges 2's 200mV 2V 10V (maybe 15V) 200V\n\nStraight in for 2V range and 200V range (scaled to 2V)\n\n200V range scaled down to 2V \n\n2V scaled allows there to be overshoot on each range, not a hard cap at 2V\n"
     (at 135.255 67.31 0)
     (effects (font (size 1.27 1.27)) (justify left bottom))
@@
     (effects (font (size 1.27 1.27)) (justify left bottom))
   )
-  (text "10V max input\n2V out\n" (at 513.715 281.305 0)
+  (text "10V range\n2V out\n" (at 500.126 282.956 0)
     (effects (font (size 1.27 1.27)) (justify left bottom))
   )
